File: pcb shield ic cmx1500ge2.sch (KiCad schematic (older format))
At the start: 13 parts, among them P1 Power, P2 Analog, P3 Digital, P4 Digital, P5 CONN_01X01, P6 CONN_01X01, P7 CONN_01X01, P8 CONN_01X01

Commit message: sampai layout pcb
Parts:
- removed J?: U.FL-R-SMT(10), symbol U.FL-R-SMT_10_:U.FL-R-SMT(10)
- added J1: SMA, Connector_Coaxial:U.FL_Molex_MCRF_73412-0110_Vertical, symbol Miscellaneous_Connectors:SMA
- added SW1: SWITCH-DPDT, Button_Switch_THT:SW_CuK_JS202011CQN_DPDT_Straight, symbol Miscellaneous_Devices:SWITCH-DPDT
- J2: renamed from J?; footprint (none) -> Connector_Coaxial:SMA_Amphenol_132289_EdgeMount
- U1: renamed from U?; footprint (none) -> modul:CXM1500GE
- gave numbers to parts that had none: 2
Connections:
- net labels added: 10(**_SS), 11(**_MOSI), A4(SDA)_l, A5(SCL)_l, RX, TX
- net labels removed: 10(**/SS), 11(**/MOSI)
- wire segments 106 -> 120
Changed lines of the file:
@@
 Text Label 10550 2600 0    60   ~ 0
 4
-Text Label 10550 2500 0    60   ~ 0
-5(**)
 Text Label 10550 2400 0    60   ~ 0
 6(**)
@@
 Text Label 10550 2000 0    60   ~ 0
 9(**)
-Text Label 10550 1900 0    60   ~ 0
-10(**/SS)
 Text Label 10550 1800 0    60   ~ 0
-11(**/MOSI)
+11(**_MOSI)
 Text Label 10550 1700 0    60   ~ 0
 12(MISO)
@@
 NoConn ~ 9400 1600
 Text Label 10550 1300 0    60   ~ 0
-A4(SDA)
+A4(SDA)_l
 Text Label 10550 1200 0    60   ~ 0
-A5(SCL)
+A5(SCL)_l
 Text Notes 10850 1000 0    60   ~ 0
 Holes
@@
 	7300 1250 7100 1250
 Wire Wire Line
-	7100 2150 7300 2150
-Wire Wire Line
 	8100 950  8100 1250
 Connection ~ 8100 1250
@@
 	7900 3150 7900 3050
 $Comp
-L modul:modul_dc-dc_lm2596 LM2596_?
+L modul:modul_dc-dc_lm2596 LM2596_1
 U 1 1 5CC48CC0
 P 7600 1050
-F 0 "LM2596_?" H 7625 1115 50  0000 C CNN
+F 0 "LM2596_1" H 7625 1115 50  0000 C CNN
 F 1 "modul_dc-dc_lm2596" H 7625 1024 50  0000 C CNN
 F 2 "modul:modul_lvl_dc-dc_lm2596" H 7600 950 50  0001 C CNN
@@
 	1    0    0    -1
 $EndComp
-$Comp
-L modul:modul_lvl-conveter_cjmcu TXS0108E-8_?
-U 1 1 5CC5751F
-P 7050 2250
-F 0 "TXS0108E-8_?" H 7600 2500 50  0000 C CNN
-F 1 "modul_lvl-conveter_cjmcu" V 7600 1900 50  0000 C CNN
-F 2 "modul:modul_lvl_conveter_cjmcu" H 7300 2550 50  0001 C CNN
-F 3 "" H 7300 2550 50  0001 C CNN
-	1    7050 2250
-	1    0    0    -1
-$EndComp
-Wire Wire Line
-	7050 2250 7300 2250
 Wire Wire Line
 	5800 700  7050 700
@@
 	7000 650  7000 2350
 Wire Wire Line
-	7000 2350 7300 2350
-Wire Wire Line
 	7050 700  7050 2250
 $Comp
-L U.FL-R-SMT_10_:U.FL-R-SMT(10) J?
-U 1 1 5CC9C483
-P 3750 2250
-F 0 "J?" H 3920 2085 50  0000 L CNN
-F 1 "U.FL-R-SMT(10)" H 3920 1994 50  0000 L CNN
-F 2 "" H 3750 2250 50  0001 L BNN
-F 3 "" H 3750 2250 50  0001 L BNN
-	1    3750 2250
-	-1   0    0    -1
-$EndComp
-$Comp
-L RF_Module:CXM1500GE U?
+L RF_Module:CXM1500GE U1
 U 1 1 5CC5C1B3
 P 5800 2550
-F 0 "U?" H 5700 4600 50  0000 C CNN
+F 0 "U1" H 5700 4600 50  0000 C CNN
 F 1 "CXM1500GE" H 5700 4500 50  0000 C CNN
-F 2 "" H 4850 3350 50  0001 C CNN
+F 2 "modul:CXM1500GE" H 4850 3350 50  0001 C CNN
 F 3 "" H 4850 3350 50  0001 C CNN
 	1    5800 2550
@@
 Wire Wire Line
 	4400 3050 4750 3050
-$Comp
-L Miscellaneous_Connectors:SMA J?
-U 1 1 5CC5EA1B
-P 4100 3050
-F 0 "J?" H 4208 3315 50  0000 C CNN
-F 1 "SMA" H 4208 3224 50  0000 C CNN
-F 2 "" H 3920 3100 60  0001 C CNN
-F 3 "" H 4100 3050 60  0000 C CNN
-	1    4100 3050
-	1    0    0    -1
-$EndComp
 Connection ~ 7100 2150
 Wire Wire Line
@@
 Wire Wire Line
 	5700 650  5700 1600
-Wire Wire Line
-	6750 2450 7300 2450
-Wire Wire Line
-	6750 2550 7300 2550
-Wire Wire Line
-	6750 2650 7300 2650
-Wire Wire Line
-	6750 2750 7300 2750
-Wire Wire Line
-	6750 2850 7300 2850
-Wire Wire Line
-	6750 2950 7300 2950
 Wire Wire Line
 	6750 3050 6900 3050
@@
 $EndComp
 Wire Wire Line
-	7300 3050 7200 3050
-Wire Wire Line
 	7200 3050 7200 3150
 $Comp
@@
 	1    0    0    -1
 $EndComp
+$Comp
+L Miscellaneous_Devices:SWITCH-DPDT SW1
+U 1 1 5CBF2FF7
+P 8450 3800
+F 0 "SW1" H 8450 4115 50  0000 C CNN
+F 1 "SWITCH-DPDT" H 8450 4024 50  0000 C CNN
+F 2 "Button_Switch_THT:SW_CuK_JS202011CQN_DPDT_Straight" H 8150 3800 60  0001 C CNN
+F 3 "" H 8450 3800 60  0000 C CNN
+	1    8450 3800
+	1    0    0    -1
+$EndComp
+Wire Wire Line
+	7900 2950 8050 2950
+Wire Wire Line
+	7900 2850 8050 2850
+Text Label 10550 2500 0    60   ~ 0
+5(**)
+Wire Wire Line
+	7900 2750 8050 2750
+Wire Wire Line
+	7900 2650 8050 2650
+Wire Wire Line
+	7900 2550 8050 2550
+Wire Wire Line
+	7900 2450 8050 2450
+Wire Wire Line
+	7900 2350 8050 2350
+Wire Wire Line
+	7900 2250 8050 2250
+Wire Wire Line
+	8100 3800 7900 3800
+Wire Wire Line
+	8100 4150 7900 4150
+Wire Wire Line
+	8800 3700 9000 3700
+Wire Wire Line
+	8800 3900 9000 3900
+Wire Wire Line
+	8800 4050 9000 4050
+Wire Wire Line
+	7300 3050 7200 3050
+Wire Wire Line
+	6750 2950 7300 2950
+Wire Wire Line
+	6750 2850 7300 2850
+Wire Wire Line
+	6750 2750 7300 2750
+Wire Wire Line
+	6750 2650 7300 2650
+Wire Wire Line
+	6750 2550 7300 2550
+Wire Wire Line
+	6750 2450 7300 2450
+Wire Wire Line
+	7000 2350 7300 2350
+Wire Wire Line
+	7050 2250 7300 2250
+Wire Wire Line
+	7100 2150 7300 2150
+$Comp
+L modul:modul_lvl-conveter_cjmcu TXS0108E-8_1
+U 1 1 5CC5751F
+P 7050 2250
+F 0 "TXS0108E-8_1" H 7600 2500 50  0000 C CNN
+F 1 "modul_lvl-conveter_cjmcu" V 7600 1900 50  0000 C CNN
+F 2 "modul:modul_lvl_conveter_cjmcu" H 7300 2550 50  0001 C CNN
+F 3 "" H 7300 2550 50  0001 C CNN
+	1    7050 2250
+	1    0    0    -1
+$EndComp
+Wire Wire Line
+	8800 4250 9000 4250
+Text Label 9000 3900 2    50   ~ 0
+1(Tx)
+Text Label 9000 4250 2    50   ~ 0
+0(Rx)
+Text Label 8050 2850 2    50   ~ 0
+TX
+Text Label 8050 2750 2    50   ~ 0
+RX
+Text Label 7900 3800 0    50   ~ 0
+RX
+Text Label 7900 4150 0    50   ~ 0
+TX
+Text Label 9000 3700 2    50   ~ 0
+8
+Text Label 9000 4050 2    50   ~ 0
+2
+Text Label 8050 2950 2    50   ~ 0
+4
+Text Label 8050 2450 0    50   ~ 0
+9(**)
+Text Label 8050 2650 0    50   ~ 0
+3(**)
+Text Label 10550 1900 0    60   ~ 0
+10(**_SS)
+Text Label 8050 2550 0    50   ~ 0
+10(**_SS)
+Text Label 8050 2250 0    50   ~ 0
+12(MISO)
+Text Label 8050 2350 0    50   ~ 0
+11(**_MOSI)
+$Comp
+L Miscellaneous_Connectors:SMA J2
+U 1 1 5CC5EA1B
+P 4100 3050
+F 0 "J2" H 4208 3315 50  0000 C CNN
+F 1 "SMA" H 4208 3224 50  0000 C CNN
+F 2 "Connector_Coaxial:SMA_Amphenol_132289_EdgeMount" H 3920 3100 60  0001 C CNN
+F 3 "" H 4100 3050 60  0001 C CNN
+	1    4100 3050
+	1    0    0    -1
+$EndComp
+$Comp
+L Miscellaneous_Connectors:SMA J1
+U 1 1 5CC050B7
+P 3850 2250
+F 0 "J1" H 3958 2515 50  0000 C CNN
+F 1 "SMA" H 3958 2424 50  0000 C CNN
+F 2 "Connector_Coaxial:U.FL_Molex_MCRF_73412-0110_Vertical" H 3670 2300 60  0001 C CNN
+F 3 "" H 3850 2250 60  0001 C CNN
+	1    3850 2250
+	1    0    0    -1
+$EndComp

Commit message: routing PCB sudah selesai
Parts:
- P1: symbol Connector_Generic:Conn_01x08 -> modul:Conn_01x08_copy
Connections:
- wire segments 120 -> 133
- no-connect marks 5 -> 34
Changed lines of the file:
@@
 Shield for Arduino that uses\nthe same pin disposition\nlike "Uno" board Rev 3.
 $Comp
-L Connector_Generic:Conn_01x08 P1
+L modul:Conn_01x08_copy P1
 U 1 1 56D70129
 P 9600 1900
@@
 	8100 2150 7900 2150
 Wire Wire Line
-	7300 1250 7100 1250
-Wire Wire Line
 	8100 950  8100 1250
 Connection ~ 8100 1250
-Text Label 7100 1250 0    50   ~ 0
-+2V
-Wire Wire Line
-	7300 1650 7600 1650
 $Comp
 L power:GND #PWR0101
 U 1 1 5CC32976
-P 7600 1650
-F 0 "#PWR0101" H 7600 1400 50  0001 C CNN
-F 1 "GND" H 7605 1477 50  0000 C CNN
-F 2 "" H 7600 1650 50  0001 C CNN
-F 3 "" H 7600 1650 50  0001 C CNN
-	1    7600 1650
-	1    0    0    -1
-$EndComp
-Connection ~ 7600 1650
-Wire Wire Line
-	7600 1650 7950 1650
+P 7600 1700
+F 0 "#PWR0101" H 7600 1450 50  0001 C CNN
+F 1 "GND" H 7605 1527 50  0000 C CNN
+F 2 "" H 7600 1700 50  0001 C CNN
+F 3 "" H 7600 1700 50  0001 C CNN
+	1    7600 1700
+	1    0    0    -1
+$EndComp
 Wire Wire Line
 	7900 3150 7900 3050
-$Comp
-L modul:modul_dc-dc_lm2596 LM2596_1
-U 1 1 5CC48CC0
-P 7600 1050
-F 0 "LM2596_1" H 7625 1115 50  0000 C CNN
-F 1 "modul_dc-dc_lm2596" H 7625 1024 50  0000 C CNN
-F 2 "modul:modul_lvl_dc-dc_lm2596" H 7600 950 50  0001 C CNN
-F 3 "" H 7600 950 50  0001 C CNN
-	1    7600 1050
-	1    0    0    -1
-$EndComp
 $Comp
 L Power:+5V #PWR0102
@@
 	5700 650  5700 1600
 Wire Wire Line
-	6750 3050 6900 3050
-Wire Wire Line
 	6900 3050 6900 3250
 $Comp
@@
 Wire Wire Line
 	7100 2150 7300 2150
-$Comp
-L modul:modul_lvl-conveter_cjmcu TXS0108E-8_1
-U 1 1 5CC5751F
-P 7050 2250
-F 0 "TXS0108E-8_1" H 7600 2500 50  0000 C CNN
-F 1 "modul_lvl-conveter_cjmcu" V 7600 1900 50  0000 C CNN
-F 2 "modul:modul_lvl_conveter_cjmcu" H 7300 2550 50  0001 C CNN
-F 3 "" H 7300 2550 50  0001 C CNN
-	1    7050 2250
-	1    0    0    -1
-$EndComp
 Wire Wire Line
 	8800 4250 9000 4250
@@
 	1    0    0    -1
 $EndComp
+Wire Wire Line
+	6650 1550 6650 1450
+Connection ~ 6650 1450
+Wire Wire Line
+	6650 1350 6650 1250
+Connection ~ 6650 1350
+Wire Wire Line
+	6650 1150 6650 1250
+Connection ~ 6650 1250
+Wire Wire Line
+	6650 1050 6650 1150
+Connection ~ 6650 1150
+Wire Wire Line
+	6650 950  6650 1050
+Connection ~ 6650 1050
+Wire Wire Line
+	6650 850  6650 950
+Connection ~ 6650 950
+Wire Wire Line
+	6200 1400 6650 1400
+Wire Wire Line
+	6650 1400 6650 1350
+Connection ~ 6200 1400
+Wire Wire Line
+	6650 1450 6650 1400
+Connection ~ 6650 1400
+Wire Wire Line
+	6750 3250 6800 3250
+Wire Wire Line
+	6800 3250 6800 3050
+Wire Wire Line
+	6750 3050 6800 3050
+Wire Wire Line
+	6800 3050 6900 3050
+Connection ~ 6800 3050
+NoConn ~ 5500 1600
+NoConn ~ 5600 1600
+NoConn ~ 5400 3700
+NoConn ~ 5500 3700
+NoConn ~ 5600 3700
+NoConn ~ 5700 3700
+NoConn ~ 5800 3700
+NoConn ~ 5900 3700
+NoConn ~ 6000 3700
+NoConn ~ 6100 3700
+NoConn ~ 6200 3700
+$Comp
+L modul:modul_dc-dc_lm2596 LM2596_1
+U 1 1 5CC48CC0
+P 7650 1050
+F 0 "LM2596_1" H 7675 1115 50  0000 C CNN
+F 1 "modul_dc-dc_lm2596" H 7675 1024 50  0000 C CNN
+F 2 "modul:modul_lvl_dc-dc_lm2596" H 7650 950 50  0001 C CNN
+F 3 "" H 7650 950 50  0001 C CNN
+	1    7650 1050
+	-1   0    0    -1
+$EndComp
+Text Label 7100 1250 0    50   ~ 0
++2V
+Wire Wire Line
+	7300 1250 7100 1250
+NoConn ~ 3850 2550
+NoConn ~ 4100 3350
+$Comp
+L modul:modul_lvl-conveter_cjmcu TXS0108E-8_1
+U 1 1 5CC5751F
+P 7050 2250
+F 0 "TXS0108E-8_1" H 7600 2500 50  0000 C CNN
+F 1 "modul_lvl-conveter_cjmcu" V 7600 1900 50  0000 C CNN
+F 2 "modul:modul_lvl_conveter_cjmcu" H 7300 2550 50  0001 C CNN
+F 3 "" H 7300 2550 50  0001 C CNN
+	1    7050 2250
+	1    0    0    -1
+$EndComp
+Wire Wire Line
+	7300 1650 7600 1650
+Wire Wire Line
+	7600 1700 7600 1650
+Connection ~ 7600 1650
+Wire Wire Line
+	7600 1650 7950 1650
+NoConn ~ 9400 2300
+NoConn ~ 9400 1700
+NoConn ~ 9400 1800
+NoConn ~ 9400 2500
+NoConn ~ 9400 2600
+NoConn ~ 9400 2700
+NoConn ~ 9400 2800
+NoConn ~ 9400 2900
+NoConn ~ 9400 3000
+NoConn ~ 10200 2300
+NoConn ~ 10200 2400
+NoConn ~ 10200 2500
+NoConn ~ 10200 1200
+NoConn ~ 10200 1300
+NoConn ~ 10200 1400
+NoConn ~ 10200 1600
 $EndSCHEMATC

Commit message: pengubahan komponen dpdt dan perbaikan routing layer pada rf komponen
Parts:
- SW1: footprint Button_Switch_THT:SW_CuK_JS202011CQN_DPDT_Straight -> Switches:Switch_DPDT_6p_TH; symbol Miscellaneous_Devices:SWITCH-DPDT -> Miscellaneous__Devices_dat:SWITCH-DPDT_V2
Connections:
- wire segments 133 -> 135
- no-connect marks 34 -> 32
Changed lines of the file:
@@
-	1    0    0    -1
-$EndComp
-$Comp
-L Miscellaneous_Devices:SWITCH-DPDT SW1
-U 1 1 5CBF2FF7
-P 8450 3800
-F 0 "SW1" H 8450 4115 50  0000 C CNN
-F 1 "SWITCH-DPDT" H 8450 4024 50  0000 C CNN
-F 2 "Button_Switch_THT:SW_CuK_JS202011CQN_DPDT_Straight" H 8150 3800 60  0001 C CNN
-F 3 "" H 8450 3800 60  0000 C CNN
-	1    8450 3800
 	1    0    0    -1
 $EndComp
@@
 Wire Wire Line
 	7300 1250 7100 1250
-NoConn ~ 3850 2550
-NoConn ~ 4100 3350
 $Comp
 L modul:modul_lvl-conveter_cjmcu TXS0108E-8_1
@@
 NoConn ~ 10200 1400
 NoConn ~ 10200 1600
+$Comp
+L power:GND #PWR0107
+U 1 1 5CC19635
+P 4100 3500
+F 0 "#PWR0107" H 4100 3250 50  0001 C CNN
+F 1 "GND" H 4105 3327 50  0000 C CNN
+F 2 "" H 4100 3500 50  0001 C CNN
+F 3 "" H 4100 3500 50  0001 C CNN
+	1    4100 3500
+	1    0    0    -1
+$EndComp
+$Comp
+L power:GND #PWR0108
+U 1 1 5CC18EDA
+P 3850 2700
+F 0 "#PWR0108" H 3850 2450 50  0001 C CNN
+F 1 "GND" H 3855 2527 50  0000 C CNN
+F 2 "" H 3850 2700 50  0001 C CNN
+F 3 "" H 3850 2700 50  0001 C CNN
+	1    3850 2700
+	1    0    0    -1
+$EndComp
+Wire Wire Line
+	3850 2550 3850 2700
+Wire Wire Line
+	4100 3350 4100 3500
+$Comp
+L Miscellaneous__Devices_dat:SWITCH-DPDT_V2 SW1
+U 1 1 5CBF2FF7
+P 8450 3800
+F 0 "SW1" H 8450 4115 50  0000 C CNN
+F 1 "SWITCH-DPDT" H 8450 4024 50  0000 C CNN
+F 2 "Switches:Switch_DPDT_6p_TH" H 8150 3800 60  0001 C CNN
+F 3 "" H 8450 3800 60  0000 C CNN
+	1    8450 3800
+	1    0    0    -1
+$EndComp
 $EndSCHEMATC

Commit message: initial commit
Parts:
- removed LM2596_1: modul_dc-dc_lm2596, modul:modul_lvl_dc-dc_lm2596, symbol modul:modul_dc-dc_lm2596
- removed P5, P6, P7, P8: CONN_01X01, Socket_Arduino_Uno:Arduino_1pin, symbol Connector_Generic:Conn_01x01
- removed SW1: SWITCH-DPDT, Switches:Switch_DPDT_6p_TH, symbol Miscellaneous__Devices_dat:SWITCH-DPDT_V2
- removed TXS0108E-8_1: modul_lvl-conveter_cjmcu, modul:modul_lvl_conveter_cjmcu, symbol modul:modul_lvl-conveter_cjmcu
- added C1, C4: 100uF, Capacitors:C_Ceramic_SMD_0603, symbol Capacitor:P-100uF_16V
- added C2, C3: 0.1u, Capacitors:C_Ceramic_SMD_0603, symbol pspice:CAP
- added C5: 10uf, Capacitors:C_Ceramic_SMD_0603, symbol Capacitor:P-10uF_6.3V
- added J3, J4: Conn_01x01_Male, Headers:Pin_Header_1x01_Male_10mil_Straight_TH, symbol Connector:Conn_01x01_Male
- added P7: Communication, Socket_Arduino_Mega:Socket_Strip_Arduino_1x08, symbol Connector_Generic:Conn_01x08
- added PB1: BUTTON, Push_Buttons:Button_4p_W-6.0mm_L-6.0mm_Normal_SMD, symbol Miscellaneous_Devices:BUTTON
- added R1: 121, Resistors:R_Chip_SMD_0603, symbol Resistor:120_0.125W
- added R2: ?, Resistors:R_Chip_SMD_0603, symbol Resistor:120_0.125W
- added R3, R4: RES, Resistors:R_Chip_SMD_0603, symbol Miscellaneous_Devices:RES
- added R5, R6: 10, Resistors:R_Chip_SMD_0603, symbol Miscellaneous_Devices:RES
- added R7, R8: -, Resistors:R_Chip_SMD_0603, symbol Resistor:120_0.125W
- added U2: TXS0108EPW, Package_SO:TSSOP-20_4.4x6.5mm_P0.65mm, symbol Logic_LevelTranslator:TXS0108EPW
- added U3: LM1117-Adj, smd:TO261AA-LM1117_rev, symbol Regulator_Linear:LM1117-ADJ
- J1: footprint Connector_Coaxial:U.FL_Molex_MCRF_73412-0110_Vertical -> Connectors_SMA:SMA_Male_Angled_TH
- J2: footprint Connector_Coaxial:SMA_Amphenol_132289_EdgeMount -> Antenna:ufl_male_smd; symbol Miscellaneous_Connectors:SMA -> U.FL-R-SMT_10_:U.FL-R-SMT(10)
- P1: symbol modul:Conn_01x08_copy -> Connector_Generic:Conn_01x08
- P2: footprint Socket_Arduino_Uno:Socket_Strip_Arduino_1x06 -> Socket_Arduino_Uno:Socket_Strip_Arduino_1x08; symbol Connector_Generic:Conn_01x06 -> Connector_Generic:Conn_01x08
- U1: footprint modul:CXM1500GE -> modul:_CXM1501GE; symbol RF_Module:CXM1500GE -> RF_Module:CXM1501GE
Connections:
- net labels added: 14(Tx3), 15(Rx3), 16(Tx2), 17(Rx2), 18(Tx1), 19(Rx1), 20(SDA), 21(SCL), 3V3, A6, A7, CTS_IC, ENB, INT_1, INT_2, RTS_IC, RX_IC, TX_IC, WK_IC
- net labels removed: +3.3V, 2, RX, TX, Vin
- wire segments 135 -> 193
- no-connect marks 32 -> 37
Other:
- note added: "Shield for Arduino Mega Rev 3"
- note removed: "Holes"
- note removed: "Shield for Arduino that uses\nthe same pin disposition\nlike "Uno" board Rev 3."
- moved on the sheet: J1, P3, P4
