File: _autosave-_autosave-pcb shield ic cmx1500ge2.kicad_pcb (KiCad board)
At the start: 2 copper layers, 72.6 x 53.4 mm, 63 parts, among them J1 SMA, J2 U.FL, J3 Conn_01x01_Male, J4 Conn_01x01_Male, J5 SMA, J6 GND, J7 VCC, J8 Conn_01x10, P1 Analog, P2 Analog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

Commit message: initial Commit
Parts:
- added ?: , , F.Cu at (135.5, 88.8)
- added J4: Conn_01x01_Male, Headers:Pin_Header_1x01_Male_10mil_Straight_TH, F.Cu at (135.3, 92.1)
- added J4: Conn_01x01_Male, Headers:Pin_Header_1x01_Male_10mil_Straight_TH, F.Cu at (135.3, 89.5)
- moved C11 2.45 mm to (147.3, 79.6)
- moved L1 1.63 mm to (147.2, 118.3)
Routing:
- net /RTS: track 8.84 -> 20.5 mm
- net /DTR: track 2.55 -> 7.03 mm
- net Net-(C14-Pad2): track 10.0 -> 7.43 mm
- net GND: track 48.2 -> 50.4 mm, vias 37 -> 59
- net /CTS_IC_L: track 11.6 -> 12.6 mm, vias 0 -> 1
- net /INT_1_L: track 12.6 -> 13.6 mm, vias 0 -> 1
- net /RX_IC_L: track 5.51 -> 6.56 mm, vias 0 -> 1
- net /TX_IC_L: track 3.44 -> 4.48 mm, vias 0 -> 1
- net /RTS_IC_L: track 5.95 -> 6.99 mm, vias 0 -> 1
- net /ENB_L: track 13.5 -> 14.6 mm, vias 0 -> 1
- net Net-(C12-Pad1): track 7.49 -> 8.33 mm
Other:
- board text added: "FS-CXM1501GR-MEGA"
- board text removed: "FS-CXM1500GR-MEGA"
